File: rioctrl-controller/rioctrl-controller.kicad_pcb (KiCad board)
At the start: 4 copper layers, 100 x 100 mm, 181 parts, among them J1 TERM-BLK-2H, J10 Conn_02x06_Odd_Even, J2 PIN_HEADER_3V, J3 TYPE-C-31-M-12, J4 Conn_02x05_Odd_Even, J5 PIN_HEADER_3V, J6 RJ45_Pulse_J0011D21BNL, J7 Conn_02x25_Odd_Even, J8 Conn_02x05_PH, J9 Conn_02x14_Odd_Even, Q1 BSS138W, Q2 BSS138W, Q3 BSS138W, SW1 SW_PUSH_SMALL, U1 TD6811, U10 W25Q16JVSS, U2 TPS54335ADDAR, U3 TPS54335ADDAR, U4 NCP114ASN250T1G, U5 W25Q16JVSS, U6 USBLC6-4SC6, U7 RP2040, U8 W5500, U9 ECP5U_45_CABGA256, X1 OSC_25MHz, Y1 Crystal_12MHz, Y2 Crystal_25MHz

Commit message: Initial schematic and layout of rioctrl-backplane
Parts:
- moved J9 0.11 mm to (135.9, 123.0)
- moved J7 0.08 mm to (186.2, 123.0)
Routing:
- net GND: vias 140 -> 210
- added copper zone on B.Cu, net GND
Other:
- board text added: "CDONE"
- board text added: "RV2024"
- board text added: "rioctrl-controller v1.0"
