File: rioctrl-controller/w5500.kicad_sch (KiCad schematic)
At the start: 34 parts, among them J6 RJ45_Pulse_J0011D21BNL, U8 W5500, Y2 Crystal_25MHz

Commit message: Fix ERC, add title information to sch, add initial version of build scripts
Other:
- company: (none) -> R. Veips
- title: (none) -> ${PROJECTNAME}
Changed lines of the file:
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@@
 	(generator_version "8.0")
 	(paper "A4")
+	(title_block
+		(title "${PROJECTNAME}")
+		(date "2024-08-25")
+		(rev "${VERSION}")
+		(company "R. Veips")
+	)
 	(junction
 		(at 175.26 78.74)

Commit message: Fill in BOM (LCSC#)
Parts:
- C33, C34: LCSC# (none) -> C92671
- C35, C39: LCSC# (none) -> C85713
- C36, C40, C41: LCSC# (none) -> C14663
- C37, C46: LCSC# (none) -> C100042
- C38: LCSC# (none) -> C1705
- C43: LCSC# (none) -> C77571
- C44, C45: LCSC# (none) -> C1631
- R24: LCSC# (none) -> C107698
- R25: LCSC# (none) -> C22865
- R29, R30, R31, R32: LCSC# (none) -> C98220
- R33, R34: LCSC# (none) -> C105881
- R35, R36, R37, R38: LCSC# (none) -> C95177
- R39, R40, R42, R43: LCSC# (none) -> C114625
- R41: LCSC# (none) -> C109318
- U8: LCSC# (none) -> C32843
