File: rioctrl-quadenc4/rioctrl-quadenc4.kicad_sch (KiCad schematic)
At the start: 0 parts

Commit message: Fix ERC, add title information to sch, add initial version of build scripts
Other:
- company: (none) -> R. Veips
- title: (none) -> rioctrl-quadenc4
Changed lines of the file:
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@@
 	(generator_version "8.0")
 	(paper "A4")
+	(title_block
+		(title "rioctrl-quadenc4")
+		(date "2024-08-25")
+		(rev "${VERSION}")
+		(company "R. Veips")
+	)
 	(no_connect
 		(at 120.65 74.93)
