File: rioctrl-shiftio/rioctrl-shiftio.kicad_pcb (KiCad board)
At the start: 2 copper layers, 100 x 100 mm, 141 parts, among them J1 Conn_02x13_Odd_Even, J2 TERM-BLK-02x05, J3 TERM-BLK-02x05, J4 TERM-BLK-02x05, J5 TERM-BLK-02x05, Q1 BSS138W, Q10 MMBT3906, Q11 AO3401A, Q12 MMBT3906, Q13 AO3401A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

Commit message: Fill in BOM (LCSC#)
Parts:
- RN1, RN2, RN3, RN4: value R_Pack04 -> 220R
