File: rioctrl-shiftio/input_shiftreg.kicad_sch (KiCad schematic)
At the start: 9 parts, among them J4 TERM-BLK-02x05, J5 TERM-BLK-02x05, U7 74HC165, U8 74HC165

Commit message: Fill in BOM (LCSC#)
Parts:
- C3, C4: LCSC# (none) -> C14663
- R53, R54, R55: LCSC# (none) -> C98220
Changed lines of the file:
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@@
 	(label "INA8"
 		(at 229.87 55.88 0)
+		(fields_autoplaced yes)
 		(effects
 			(font
@@
 	(label "INA6"
 		(at 229.87 53.34 0)
+		(fields_autoplaced yes)
 		(effects
 			(font
@@
 	(label "INA1"
 		(at 210.82 48.26 0)
+		(fields_autoplaced yes)
 		(effects
 			(font
@@
 	(label "INA2"
 		(at 229.87 48.26 0)
+		(fields_autoplaced yes)
 		(effects
 			(font
@@
 	(label "INA1"
 		(at 182.88 44.45 0)
+		(fields_autoplaced yes)
 		(effects
 			(font
@@
 	(label "INA4"
 		(at 229.87 50.8 0)
+		(fields_autoplaced yes)
 		(effects
 			(font
@@
 			)
 		)
+		(property "LCSC#" "C98220"
+			(at 127 80.01 0)
+			(effects
+				(font
+					(size 1.27 1.27)
+				)
+				(hide yes)
+			)
+		)
 		(pin "1"
 		)
@@
 		)
 		(property "Description" "Resistor, small symbol"
+			(at 127 158.75 0)
+			(effects
+				(font
+					(size 1.27 1.27)
+				)
+				(hide yes)
+			)
+		)
+		(property "LCSC#" "C98220"
 			(at 127 158.75 0)
 			(effects
@@
 			)
 		)
+		(property "LCSC#" "C14663"
+			(at 101.6 27.94 0)
+			(effects
+				(font
+					(size 1.27 1.27)
+				)
+				(hide yes)
+			)
+		)
 		(pin "1"
 		)
@@
 		)
 		(property "Description" "Resistor, small symbol"
+			(at 132.08 119.38 0)
+			(effects
+				(font
+					(size 1.27 1.27)
+				)
+				(hide yes)
+			)
+		)
+		(property "LCSC#" "C98220"
 			(at 132.08 119.38 0)
 			(effects
@@
 			(at 101.6 106.68 0)
 			(effects
+				(font
+					(size 1.27 1.27)
+				)
+				(hide yes)
+			)
+		)
+		(property "LCSC#" "C14663"
+			(at 101.6 106.68 0)
+			(effects

Commit message: Regenerate outputs with more 3D models
Parts:
- J4, J5: MatingLCSC# (none) -> C2908401
Changed lines of the file:
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@@
+			)
+		)
+		(property "MatingLCSC#" "C2908401"
+			(at 220.98 129.54 0)
+			(effects
+				(font
+					(size 1.27 1.27)
+				)
+				(hide yes)
 			)
 		)
@@
 			(at 220.98 50.8 0)
 			(effects
+				(font
+					(size 1.27 1.27)
+				)
+				(hide yes)
+			)
+		)
+		(property "MatingLCSC#" "C2908401"
+			(at 220.98 50.8 0)
+			(effects
