File: rioctrl-shiftio/out_shiftreg.kicad_sch (KiCad schematic)
At the start: 8 parts, among them J2 TERM-BLK-02x05, J3 TERM-BLK-02x05, U1 74HC595, U2 74HC595

Commit message: Fill in BOM (LCSC#)
Parts:
- C1, C2: LCSC# (none) -> C14663
- R3, R4: LCSC# (none) -> C98220
Changed lines of the file:
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@@
+			)
+		)
+		(property "LCSC#" "C14663"
+			(at 121.92 31.75 0)
+			(effects
+				(font
+					(size 1.27 1.27)
+				)
+				(hide yes)
 			)
 		)
@@
 			)
 		)
+		(property "LCSC#" "C98220"
+			(at 72.39 119.38 0)
+			(effects
+				(font
+					(size 1.27 1.27)
+				)
+				(hide yes)
+			)
+		)
 		(pin "1"
 		)
@@
 			)
 		)
+		(property "LCSC#" "C98220"
+			(at 72.39 50.8 0)
+			(effects
+				(font
+					(size 1.27 1.27)
+				)
+				(hide yes)
+			)
+		)
 		(pin "1"
 		)
@@
 			(at 121.92 100.33 0)
 			(effects
+				(font
+					(size 1.27 1.27)
+				)
+				(hide yes)
+			)
+		)
+		(property "LCSC#" "C14663"
+			(at 121.92 100.33 0)
+			(effects

Commit message: Regenerate outputs with more 3D models
Parts:
- J2, J3: MatingLCSC# (none) -> C2908401
Changed lines of the file:
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@@
+			)
+		)
+		(property "MatingLCSC#" "C2908401"
+			(at 208.28 123.19 0)
+			(effects
+				(font
+					(size 1.27 1.27)
+				)
+				(hide yes)
 			)
 		)
@@
 			(at 208.28 54.61 0)
 			(effects
+				(font
+					(size 1.27 1.27)
+				)
+				(hide yes)
+			)
+		)
+		(property "MatingLCSC#" "C2908401"
+			(at 208.28 54.61 0)
+			(effects
