File: rioctrl-shiftio/digital_output.kicad_sch (KiCad schematic)
At the start: 6 parts, among them Q26 MMBT3906, Q27 AO3401A

Commit message: Fill in BOM (LCSC#)
Parts:
- R41: LCSC# (none) -> C105579
- R42: LCSC# (none) -> C98220
- R43: LCSC# (none) -> C112305
Changed lines of the file:
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@@
+			)
+		)
+		(property "LCSC#" "C105579"
+			(at 100.33 40.64 0)
+			(effects
+				(font
+					(size 1.27 1.27)
+				)
+				(hide yes)
 			)
 		)
@@
 			)
 		)
+		(property "LCSC#" "C112305"
+			(at 118.11 31.75 0)
+			(effects
+				(font
+					(size 1.27 1.27)
+				)
+				(hide yes)
+			)
+		)
 		(pin "2"
 		)
@@
 			(at 102.87 55.88 0)
 			(effects
+				(font
+					(size 1.27 1.27)
+				)
+				(hide yes)
+			)
+		)
+		(property "LCSC#" "C98220"
+			(at 102.87 55.88 0)
+			(effects

Commit message: rioctrl-shiftio: change the part number of 1 ohm resistor (previously, an 0603 resistor was specified for 0805 footprint)
Parts:
- R43: LCSC# C112305 -> C131397
Changed lines of the file:
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@@
 			)
 		)
-		(property "LCSC#" "C112305"
+		(property "LCSC#" "C131397"
 			(at 118.11 31.75 0)
 			(effects
