File: rioctrl-stepdir4/rioctrl-stepdir4.kicad_pcb (KiCad board)
At the start: 2 copper layers, 100 x 100 mm, 93 parts, among them J1 Conn_02x13_Odd_Even, J2 RJ45_LED_Shielded, J3 RJ45_LED_Shielded, J4 RJ45_LED_Shielded, J5 RJ45_LED_Shielded, Q1 BSS138W, Q10 AO3401A, Q11 BSS138W, Q12 AO3401A, Q2 BSS138W, Q3 AO3401A, Q4 AO3401A, Q5 BSS138W, Q6 AO3401A, Q7 BSS138W, Q8 AO3401A, Q9 BSS138W, U1 CS48505S, U10 CS48505S, U11 CS48505S, U12 USBLC6-4SC6, U2 CS48505S, U3 USBLC6-4SC6, U4 CS48505S, U5 CS48505S, U6 USBLC6-4SC6, U7 CS48505S, U8 CS48505S, U9 USBLC6-4SC6

Commit message: rioctrl-stepdir4: pass ERC and DRC
Parts:
- moved Q3 0.25 mm to (118.2, 139.0)
Routing:
- net +5V: track 327.7 -> 315.4 mm
- net +24V_EN: track 224.9 -> 222.7 mm
- net GND: vias 112 -> 110
Other:
- board text added: "GND"
- board text added: "RV2024"
- board text added: "S11 S5"
- board text added: "S6 S0"
- board text added: "rioctrl-stepdir v1.0"

Commit message: Label axes on stepdir
Connections:
- net /Step dir output 0/DIR_OUT_N renamed /Step dir output 4/DIR_OUT_N
- net /Step dir output 0/DIR_OUT_P renamed /Step dir output 4/DIR_OUT_P
- net /Step dir output 0/DIR_OUT_P_N renamed /Step dir output 4/DIR_OUT_P_N
- net /Step dir output 0/DIR_OUT_P_P renamed /Step dir output 4/DIR_OUT_P_P
- net /Step dir output 0/EN_OUT renamed /Step dir output 4/EN_OUT
- net /Step dir output 0/STEP_OUT_N renamed /Step dir output 4/STEP_OUT_N
- net /Step dir output 0/STEP_OUT_P renamed /Step dir output 4/STEP_OUT_P
- net /Step dir output 0/STEP_OUT_P_N renamed /Step dir output 4/STEP_OUT_P_N
- net /Step dir output 0/STEP_OUT_P_P renamed /Step dir output 4/STEP_OUT_P_P
- F2 pad 2: /Step dir output 1/EN_OUT -> /Step dir output 3/EN_OUT
- F4 pad 2: /Step dir output 3/EN_OUT -> /Step dir output 1/EN_OUT
- J3 pad 1: /Step dir output 1/STEP_OUT_P_P -> /Step dir output 3/STEP_OUT_P_P
- J3 pad 10: /Step dir output 1/EN_OUT -> /Step dir output 3/EN_OUT
- J3 pad 2: /Step dir output 1/STEP_OUT_P_N -> /Step dir output 3/STEP_OUT_P_N
- J3 pad 3: /Step dir output 1/DIR_OUT_P_P -> /Step dir output 3/DIR_OUT_P_P
- J3 pad 4: /Step dir output 1/EN_OUT -> /Step dir output 3/EN_OUT
- J3 pad 6: /Step dir output 1/DIR_OUT_P_N -> /Step dir output 3/DIR_OUT_P_N
- J5 pad 1: /Step dir output 3/STEP_OUT_P_P -> /Step dir output 1/STEP_OUT_P_P
- J5 pad 10: /Step dir output 3/EN_OUT -> /Step dir output 1/EN_OUT
- J5 pad 2: /Step dir output 3/STEP_OUT_P_N -> /Step dir output 1/STEP_OUT_P_N
- J5 pad 3: /Step dir output 3/DIR_OUT_P_P -> /Step dir output 1/DIR_OUT_P_P
- J5 pad 4: /Step dir output 3/EN_OUT -> /Step dir output 1/EN_OUT
- J5 pad 6: /Step dir output 3/DIR_OUT_P_N -> /Step dir output 1/DIR_OUT_P_N
- R16 pad 1: /Step dir output 1/DIR_OUT_P -> /Step dir output 3/DIR_OUT_P
- R16 pad 2: /Step dir output 1/DIR_OUT_P_P -> /Step dir output 3/DIR_OUT_P_P
- R17 pad 1: /Step dir output 1/DIR_OUT_N -> /Step dir output 3/DIR_OUT_N
- R17 pad 2: /Step dir output 1/DIR_OUT_P_N -> /Step dir output 3/DIR_OUT_P_N
- R18 pad 1: /Step dir output 1/STEP_OUT_P -> /Step dir output 3/STEP_OUT_P
- R18 pad 2: /Step dir output 1/STEP_OUT_P_P -> /Step dir output 3/STEP_OUT_P_P
- R19 pad 1: /Step dir output 1/STEP_OUT_N -> /Step dir output 3/STEP_OUT_N
- R19 pad 2: /Step dir output 1/STEP_OUT_P_N -> /Step dir output 3/STEP_OUT_P_N
- R32 pad 1: /Step dir output 3/DIR_OUT_P -> /Step dir output 1/DIR_OUT_P
- R32 pad 2: /Step dir output 3/DIR_OUT_P_P -> /Step dir output 1/DIR_OUT_P_P
- R33 pad 1: /Step dir output 3/DIR_OUT_N -> /Step dir output 1/DIR_OUT_N
- R33 pad 2: /Step dir output 3/DIR_OUT_P_N -> /Step dir output 1/DIR_OUT_P_N
- R34 pad 1: /Step dir output 3/STEP_OUT_P -> /Step dir output 1/STEP_OUT_P
- R34 pad 2: /Step dir output 3/STEP_OUT_P_P -> /Step dir output 1/STEP_OUT_P_P
- R35 pad 1: /Step dir output 3/STEP_OUT_N -> /Step dir output 1/STEP_OUT_N
- R35 pad 2: /Step dir output 3/STEP_OUT_P_N -> /Step dir output 1/STEP_OUT_P_N
- U10 pad 6: /Step dir output 3/STEP_OUT_P -> /Step dir output 1/STEP_OUT_P
- U10 pad 7: /Step dir output 3/STEP_OUT_N -> /Step dir output 1/STEP_OUT_N
- U11 pad 6: /Step dir output 3/DIR_OUT_P -> /Step dir output 1/DIR_OUT_P
- U11 pad 7: /Step dir output 3/DIR_OUT_N -> /Step dir output 1/DIR_OUT_N
- U12 pad 1: /Step dir output 3/STEP_OUT_N -> /Step dir output 1/STEP_OUT_N
- U12 pad 3: /Step dir output 3/STEP_OUT_P -> /Step dir output 1/STEP_OUT_P
- U12 pad 4: /Step dir output 3/DIR_OUT_N -> /Step dir output 1/DIR_OUT_N
- U12 pad 6: /Step dir output 3/DIR_OUT_P -> /Step dir output 1/DIR_OUT_P
- U4 pad 6: /Step dir output 1/STEP_OUT_P -> /Step dir output 3/STEP_OUT_P
- U4 pad 7: /Step dir output 1/STEP_OUT_N -> /Step dir output 3/STEP_OUT_N
- U5 pad 6: /Step dir output 1/DIR_OUT_P -> /Step dir output 3/DIR_OUT_P
- U5 pad 7: /Step dir output 1/DIR_OUT_N -> /Step dir output 3/DIR_OUT_N
- U6 pad 1: /Step dir output 1/STEP_OUT_N -> /Step dir output 3/STEP_OUT_N
- U6 pad 3: /Step dir output 1/STEP_OUT_P -> /Step dir output 3/STEP_OUT_P
- U6 pad 4: /Step dir output 1/DIR_OUT_N -> /Step dir output 3/DIR_OUT_N
- U6 pad 6: /Step dir output 1/DIR_OUT_P -> /Step dir output 3/DIR_OUT_P
Routing:
- net /Step dir output 3/DIR_OUT_P_P: track 19.1 -> 20.6 mm
- net /Step dir output 1/DIR_OUT_P_P: track 20.6 -> 19.1 mm
- net /Step dir output 3/STEP_OUT_P_P: track 12.9 -> 13.8 mm
- net /Step dir output 1/STEP_OUT_P_P: track 13.8 -> 12.9 mm
Other:
- board text added: "Axis 1"
- board text added: "Axis 2"
- board text added: "Axis 3"
- board text added: "Axis 4"

Commit message: Add rioctrl-quadenc4 initial design
Routing:
- net GND: vias 110 -> 125
Other:
- board text added: "https://github.com/festlv/rioctrl-hw"
Changed lines of the file:
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@@
 		)
 	)
+	(gr_text "https://github.com/festlv/rioctrl-hw"
+		(at 114.463094 119 0)
+		(layer "F.SilkS")
+		(effects
+			(font
+				(size 1 1)
+				(thickness 0.25)
+				(bold yes)
+			)
+			(justify left bottom)
+		)
+	)
 	(gr_text "rioctrl-stepdir v1.0"
-		(at 111.2 115.2 0)
+		(at 113.742857 115.2 0)
 		(layer "F.SilkS")
 		(effects
@@
 	)
 	(via
+		(at 157.5 81)
+		(size 0.6)
+		(drill 0.3)
+		(layers "F.Cu" "B.Cu")
+		(free yes)
+		(net 1)
+	)
+	(via
 		(at 149.9 73.5)
 		(size 0.6)
@@
 	)
 	(via
+		(at 102 83)
+		(size 0.6)
+		(drill 0.3)
+		(layers "F.Cu" "B.Cu")
+		(free yes)
+		(net 1)
+	)
+	(via
 		(at 156.4 123.8)
 		(size 0.6)
@@
 	)
 	(via
+		(at 135.5 77)
+		(size 0.6)
+		(drill 0.3)
+		(layers "F.Cu" "B.Cu")
+		(free yes)
+		(net 1)
+	)
+	(via
 		(at 93.3 68.7)
 		(size 0.6)
@@
 	)
 	(via
+		(at 143 77.5)
+		(size 0.6)
+		(drill 0.3)
+		(layers "F.Cu" "B.Cu")
+		(free yes)
+		(net 1)
+	)
+	(via
 		(at 142.1 113.3)
 		(size 0.6)
@@
 	)
 	(via
+		(at 164.5 85.5)
+		(size 0.6)
+		(drill 0.3)
+		(layers "F.Cu" "B.Cu")
+		(free yes)
+		(net 1)
+	)
+	(via
 		(at 80.2 65.8)
 		(size 0.6)
@@
 	)
 	(via
+		(at 163 78)
+		(size 0.6)
+		(drill 0.3)
+		(layers "F.Cu" "B.Cu")
+		(free yes)
+		(net 1)
+	)
+	(via
 		(at 87.2 142)
 		(size 0.6)
@@
 	)
 	(via
+		(at 111.5 77.5)
+		(size 0.6)
+		(drill 0.3)
+		(layers "F.Cu" "B.Cu")
+		(free yes)
+		(net 1)
+	)
+	(via
 		(at 159.5 99.8)
 		(size 0.6)
@@
 	)
 	(via
+		(at 93 77.5)
+		(size 0.6)
+		(drill 0.3)
+		(layers "F.Cu" "B.Cu")
+		(free yes)
+		(net 1)
+	)
+	(via
 		(at 99.3 85.5)
 		(size 0.6)
@@
 	)
 	(via
+		(at 147 78)
+		(size 0.6)
+		(drill 0.3)
+		(layers "F.Cu" "B.Cu")
+		(free yes)
+		(net 1)
+	)
+	(via
 		(at 154.3 94.6)
 		(size 0.6)
@@
 	)
 	(via
+		(at 117 77.5)
+		(size 0.6)
+		(drill 0.3)
+		(layers "F.Cu" "B.Cu")
+		(free yes)
+		(net 1)
+	)
+	(via
+		(at 136 81.5)
+		(size 0.6)
+		(drill 0.3)
+		(layers "F.Cu" "B.Cu")
+		(free yes)
+		(net 1)
+	)
+	(via
 		(at 136.1 138.8)
 		(size 0.6)
@@
 	)
 	(via
+		(at 115.5 81)
+		(size 0.6)
+		(drill 0.3)
+		(layers "F.Cu" "B.Cu")
+		(free yes)
+		(net 1)
+	)
+	(via
 		(at 134.1 121.1)
 		(size 0.6)
@@
 	)
 	(via
+		(at 123 78.5)
+		(size 0.6)
+		(drill 0.3)
+		(layers "F.Cu" "B.Cu")
+		(free yes)
+		(net 1)
+	)
+	(via
 		(at 154.4 99.6)
 		(size 0.6)
@@
 	)
 	(via
+		(at 154 78)
+		(size 0.6)
+		(drill 0.3)
+		(layers "F.Cu" "B.Cu")
+		(free yes)
+		(net 1)
+	)
+	(via
 		(at 85 73.4)
 		(size 0.6)
@@
 		(net 1)
 	)
+	(via
+		(at 100.5 78)
+		(size 0.6)
+		(drill 0.3)
+		(layers "F.Cu" "B.Cu")
+		(free yes)
+		(net 1)
+	)
