File: rioctrl-spindle/rioctrl-spindle.kicad_pcb (KiCad board)
At the start: 2 copper layers, 100 x 100 mm, 121 parts, among them J1 RJ45_LED_Shielded, J2 Conn_02x13_Odd_Even, J3 RJ45_LED_Shielded, J4 RJ45_LED_Shielded, J5 RJ45_LED_Shielded, U1 CS48505S, U10 USBLC6-4SC6, U11 CS48505S, U12 CS48505S, U13 CS48505S, U14 USBLC6-4SC6, U15 USBLC6-4SC6, U16 CS48505S, U17 CS48505S, U18 CS48505S, U19 USBLC6-4SC6, U2 CS48505S, U20 USBLC6-4SC6, U3 CS48505S, U4 USBLC6-4SC6, U5 USBLC6-4SC6, U6 CS48505S, U7 CS48505S, U8 CS48505S, U9 USBLC6-4SC6

Commit message: rioctrl-spindle v1.0 release
Parts:
- removed C10, C11: 0.1uF, Capacitor_SMD:C_0603_1608Metric
- removed C12: 10uF, Capacitor_SMD:C_0805_2012Metric
- removed D3, D5: BSD5C031V, Diode_SMD:D_SOD-523
- removed D6: PESD5V0S1BBN, Diode_SMD:D_SOD-523
- removed FB2, FB3: FB_100R_3A, Inductor_SMD:L_0603_1608Metric
- removed J3, J4: RJ45_LED_Shielded, hadv-connectors:R-RJ45R08P-C000
- removed R33, R35, R36, R38, R39, R41: 1K, Resistor_SMD:R_0603_1608Metric
- removed R34, R37, R40: 120R, Resistor_SMD:R_0603_1608Metric
- removed R42, R43, R44, R45, R46, R47: 10R, Resistor_SMD:R_0603_1608Metric
- removed R48: 0R, Resistor_SMD:R_0603_1608Metric
- removed U10, U14, U15, U9: USBLC6-4SC6, Package_TO_SOT_SMD:SOT-23-6
- removed U11, U12, U13, U7, U8: CS48505S, Package_SO:SOIC-8_3.9x4.9mm_P1.27mm
- C4, C8: value 10uF -> 3.3nF; footprint Capacitor_SMD:C_0805_2012Metric -> Capacitor_SMD:C_0603_1608Metric
- C5: value 0.1uF -> 10uF
- C7, C9: value 0.1uF -> 10nF
- D2, D4: value PESD5V0S1BBN -> SMAJ10A; footprint Diode_SMD:D_SOD-523 -> Diode_SMD:D_SMA
- J1: value RJ45_LED_Shielded -> TERM-BLK-02x05; footprint hadv-connectors:R-RJ45R08P-C000 -> hadv-connectors:JL15EDGRHC-35005B02
- R10: value 10R -> 120R
- R11: value 10R -> 1K
- R16: value 0R -> 1K
- R17, R7: value 1K -> 120R
- R18, R8: value 120R -> 1K
- R19, R20, R3, R4: value 1K -> 10R
- R2, R5: value 120R -> 10R
- R21, R24: value 120R -> 10K
- R22, R23: value 1K -> 10K
- R25: value 1K -> 100K
- R26: value 10R -> 50R
- R27, R29, R30, R31: value 10R -> 10K
- R28: value 10R -> 100K
- R32: value 0R -> 50R
- U6: value CS48505S -> LM358DT; footprint Package_SO:SOIC-8_3.9x4.9mm_P1.27mm -> Package_SO:SO-8_3.9x4.9mm_P1.27mm
- moved R3 43.8 mm to (190.4, 122.0)
- moved R1 42.7 mm to (188.8, 122.0)
- moved U4 42.7 mm to (195.0, 109.3), turned to 180 degrees
- moved R2 41.7 mm to (186.2, 122.0), turned to 90 degrees
- moved FB1 39.5 mm to (156.4, 79.2), turned to 0 degrees
- moved D1 38.6 mm to (182.8, 113.5), turned to -90 degrees
- moved C4 38.0 mm to (164.6, 86.2), turned to -90 degrees
- moved R12 36.9 mm to (188.7, 106.5)
- moved R13 36.7 mm to (186.9, 106.5)
- moved D2 34.0 mm to (160.2, 65.8), turned to 180 degrees
- moved R8 31.6 mm to (185.2, 110.0), turned to -90 degrees
- moved R7 31.3 mm to (187.8, 109.2), turned to 0 degrees
- moved U1 31.1 mm to (188.1, 115.6)
- moved R6 30.7 mm to (190.6, 110.0)
- moved C1 30.7 mm to (184.6, 113.6)
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Connections:
- C4 pad 1: +5V -> Net-(U6A-+)
- C5 pad 1: +3V3 -> Net-(U6C-V+)
- C6 pad 1: +3V3 -> Net-(U6C-V+)
- C7 pad 1: +3V3 -> Net-(C7-Pad1)
- C7 pad 2: GND -> Net-(D4-A1)
- C8 pad 1: +5V -> Net-(U6B-+)
- C9 pad 1: +3V3 -> Net-(C9-Pad1)
- C9 pad 2: GND -> Net-(D2-A1)
- D2 pad 1: GND -> Net-(D2-A1)
- D2 pad 2: +5V -> GND
- D4 pad 1: GND -> Net-(D4-A1)
- D4 pad 2: +5V -> GND
- FB1 pad 1: +5V -> +24V
- FB1 pad 2: Net-(FB1-Pad2) -> Net-(U6C-V+)
- J1 pad 1: Net-(J1-Pad1) -> unconnected-(J1-Pin_1-Pad1)
- J1 pad 10: unconnected-(J1-Pad10) -> GND
- J1 pad 2: Net-(J1-Pad2) -> /Serial/SSERIAL_RX_B
- J1 pad 3: Net-(J1-Pad3) -> /Serial/MODBUS_B
- J1 pad 4: Net-(J1-Pad4) -> /Serial/SSERIAL_RX_A
- J1 pad 5: Net-(J1-Pad5) -> /Serial/MODBUS_A
- J1 pad 6: Net-(J1-Pad6) -> /Serial/SSERIAL_TX_B
- J1 pad 7: Net-(FB1-Pad2) -> /Analog outputs/AO_1
- J1 pad 8: GND -> /Serial/SSERIAL_TX_A
- J1 pad 9: unconnected-(J1-Pad9) -> /Analog outputs/AO_0
- J2 pad 10: /Quadenc3/Z -> /Quadenc/Z
- J2 pad 11: /Quadenc1/B -> /Serial/MODBUS_TX
- J2 pad 12: /Quadenc3/B -> /Quadenc/B
- J2 pad 13: /Quadenc1/A -> /Serial/MODBUS_RX
- J2 pad 14: /Quadenc3/A -> /Quadenc/A
- J2 pad 3: /Quadenc/Z -> /Analog outputs/PWM_A0
- J2 pad 4: /Quadenc2/Z -> /Serial/MODBUS_TXEN
- J2 pad 5: /Quadenc/B -> /Analog outputs/PWM_A1
- J2 pad 6: /Quadenc2/B -> /Serial/SSERIAL_TX
- J2 pad 7: /Quadenc/A -> /Slot/S2
- J2 pad 8: /Quadenc2/A -> /Serial/SSERIAL_RX
- J2 pad 9: /Quadenc1/Z -> /Slot/S3
- R1 pad 1: +3V3 -> Net-(U1-DE)
- R1 pad 2: /Quadenc/B_IN_P -> /Serial/MODBUS_TXEN
- R10 pad 1: /Quadenc/A_IN_P -> /Serial/RX_B
- R10 pad 2: Net-(J1-Pad1) -> /Serial/RX_A
- R11 pad 1: /Quadenc/A_IN_N -> /Serial/RX_B
- R11 pad 2: Net-(J1-Pad2) -> GND
- R12 pad 1: /Quadenc/B_IN_P -> Net-(U1-A)
- R12 pad 2: Net-(J1-Pad3) -> /Serial/MODBUS_A
- R13 pad 1: /Quadenc/Z_IN_P -> Net-(U1-B)
- R13 pad 2: Net-(J1-Pad4) -> /Serial/MODBUS_B
- R14 pad 1: /Quadenc/Z_IN_N -> /Serial/RX_A
- R14 pad 2: Net-(J1-Pad5) -> /Serial/SSERIAL_RX_A
- R15 pad 1: /Quadenc/B_IN_N -> /Serial/RX_B
- R15 pad 2: Net-(J1-Pad6) -> /Serial/SSERIAL_RX_B
- R16 pad 1: Net-(J1-PadSH) -> +3V3
- R16 pad 2: GND -> /Serial/TX_A
- R17 pad 1: +3V3 -> /Serial/TX_B
- R17 pad 2: /Quadenc1/B_IN_P -> /Serial/TX_A
- R18 pad 1: /Quadenc1/B_IN_P -> /Serial/TX_B
- R18 pad 2: /Quadenc1/B_IN_N -> GND
- R19 pad 1: /Quadenc1/B_IN_N -> /Serial/TX_A
- R19 pad 2: GND -> /Serial/SSERIAL_TX_A
- R2 pad 1: /Quadenc/B_IN_P -> /Serial/MODBUS_RX
- R2 pad 2: /Quadenc/B_IN_N -> Net-(U1-RO)
- R20 pad 1: +3V3 -> /Serial/TX_B
- R20 pad 2: /Quadenc1/Z_IN_P -> /Serial/SSERIAL_TX_B
- R21 pad 1: /Quadenc1/Z_IN_P -> /Analog outputs/PWM_A0
- R21 pad 2: /Quadenc1/Z_IN_N -> Net-(C7-Pad1)
- R22 pad 1: /Quadenc1/Z_IN_N -> Net-(U6A--)
- R22 pad 2: GND -> Net-(R22-Pad2)
- R23 pad 1: +3V3 -> Net-(D4-A1)
- R23 pad 2: /Quadenc1/A_IN_P -> Net-(R22-Pad2)
- R24 pad 1: /Quadenc1/A_IN_N -> GND
- R24 pad 2: /Quadenc1/A_IN_P -> Net-(U6A--)
- R25 pad 1: /Quadenc1/A_IN_N -> Net-(C7-Pad1)
- R25 pad 2: GND -> Net-(U6A-+)
- R26 pad 1: /Quadenc1/A_IN_P -> Net-(D4-A1)
- R26 pad 2: Net-(J3-Pad1) -> /Analog outputs/AO_0
- R27 pad 1: /Quadenc1/A_IN_N -> /Analog outputs/PWM_A1
- R27 pad 2: Net-(J3-Pad2) -> Net-(C9-Pad1)
- R28 pad 1: /Quadenc1/B_IN_P -> Net-(C9-Pad1)
- R28 pad 2: Net-(J3-Pad3) -> Net-(U6B-+)
- R29 pad 1: /Quadenc1/Z_IN_P -> GND
- R29 pad 2: Net-(J3-Pad4) -> Net-(U6B--)
- R3 pad 1: /Quadenc/B_IN_N -> /Serial/MODBUS_TX
- R3 pad 2: GND -> Net-(U1-DI)
- R30 pad 1: /Quadenc1/Z_IN_N -> Net-(U6B--)
- R30 pad 2: Net-(J3-Pad5) -> Net-(R30-Pad2)
- R31 pad 1: /Quadenc1/B_IN_N -> Net-(D2-A1)
- R31 pad 2: Net-(J3-Pad6) -> Net-(R30-Pad2)
- R32 pad 1: Net-(J3-PadSH) -> Net-(D2-A1)
- R32 pad 2: GND -> /Analog outputs/AO_1
- R4 pad 1: +3V3 -> /Serial/SSERIAL_RX
- R4 pad 2: /Quadenc/Z_IN_P -> Net-(U2-RO)
- R49 pad 2: /Quadenc3/B_IN_P -> /Quadenc/B_IN_P
- R5 pad 1: /Quadenc/Z_IN_P -> /Serial/SSERIAL_TX
- R5 pad 2: /Quadenc/Z_IN_N -> Net-(U3-DI)
- R50 pad 1: /Quadenc3/B_IN_P -> /Quadenc/B_IN_P
- R50 pad 2: /Quadenc3/B_IN_N -> /Quadenc/B_IN_N
- R51 pad 1: /Quadenc3/B_IN_N -> /Quadenc/B_IN_N
- R52 pad 2: /Quadenc3/Z_IN_P -> /Quadenc/Z_IN_P
- R53 pad 1: /Quadenc3/Z_IN_P -> /Quadenc/Z_IN_P
- R53 pad 2: /Quadenc3/Z_IN_N -> /Quadenc/Z_IN_N
- R54 pad 1: /Quadenc3/Z_IN_N -> /Quadenc/Z_IN_N
- R55 pad 2: /Quadenc3/A_IN_P -> /Quadenc/A_IN_P
- R56 pad 1: /Quadenc3/A_IN_N -> /Quadenc/A_IN_N
- R56 pad 2: /Quadenc3/A_IN_P -> /Quadenc/A_IN_P
- R57 pad 1: /Quadenc3/A_IN_N -> /Quadenc/A_IN_N
- R58 pad 1: /Quadenc3/A_IN_P -> /Quadenc/A_IN_P
- R59 pad 1: /Quadenc3/A_IN_N -> /Quadenc/A_IN_N
- R6 pad 1: /Quadenc/Z_IN_N -> +3V3
- R6 pad 2: GND -> Net-(U1-A)
- R60 pad 1: /Quadenc3/B_IN_P -> /Quadenc/B_IN_P
- R61 pad 1: /Quadenc3/Z_IN_P -> /Quadenc/Z_IN_P
- R62 pad 1: /Quadenc3/Z_IN_N -> /Quadenc/Z_IN_N
- R63 pad 1: /Quadenc3/B_IN_N -> /Quadenc/B_IN_N
- R7 pad 1: +3V3 -> Net-(U1-B)
- R7 pad 2: /Quadenc/A_IN_P -> Net-(U1-A)
- R8 pad 1: /Quadenc/A_IN_N -> Net-(U1-B)
- R8 pad 2: /Quadenc/A_IN_P -> GND
- R9 pad 1: /Quadenc/A_IN_N -> +3V3
- R9 pad 2: GND -> /Serial/RX_A
- U1 pad 1: /Quadenc/B -> Net-(U1-RO)
- U1 pad 2: GND -> Net-(U1-DE)
- U1 pad 3: GND -> Net-(U1-DE)
- U1 pad 4: unconnected-(U1-DI-Pad4) -> Net-(U1-DI)
- U1 pad 6: /Quadenc/B_IN_P -> Net-(U1-A)
- U1 pad 7: /Quadenc/B_IN_N -> Net-(U1-B)
- U16 pad 1: /Quadenc3/B -> /Quadenc/B
- U16 pad 6: /Quadenc3/B_IN_P -> /Quadenc/B_IN_P
- U16 pad 7: /Quadenc3/B_IN_N -> /Quadenc/B_IN_N
- U17 pad 1: /Quadenc3/Z -> /Quadenc/Z
- U17 pad 6: /Quadenc3/Z_IN_P -> /Quadenc/Z_IN_P
- U17 pad 7: /Quadenc3/Z_IN_N -> /Quadenc/Z_IN_N
- U18 pad 1: /Quadenc3/A -> /Quadenc/A
- U18 pad 6: /Quadenc3/A_IN_P -> /Quadenc/A_IN_P
- U18 pad 7: /Quadenc3/A_IN_N -> /Quadenc/A_IN_N
- U19 pad 1: /Quadenc3/A_IN_N -> /Quadenc/A_IN_N
- U19 pad 3: /Quadenc3/A_IN_P -> /Quadenc/A_IN_P
- U19 pad 4: /Quadenc3/B_IN_N -> /Quadenc/B_IN_N
- U19 pad 6: /Quadenc3/B_IN_P -> /Quadenc/B_IN_P
- U2 pad 1: /Quadenc/Z -> Net-(U2-RO)
- U2 pad 6: /Quadenc/Z_IN_P -> /Serial/RX_A
- U2 pad 7: /Quadenc/Z_IN_N -> /Serial/RX_B
- U20 pad 4: /Quadenc3/Z_IN_N -> /Quadenc/Z_IN_N
- U20 pad 6: /Quadenc3/Z_IN_P -> /Quadenc/Z_IN_P
- U3 pad 1: /Quadenc/A -> unconnected-(U3-RO-Pad1)
- U3 pad 2: GND -> +3V3
- U3 pad 3: GND -> +3V3
- U3 pad 4: unconnected-(U3-DI-Pad4) -> Net-(U3-DI)
- U3 pad 6: /Quadenc/A_IN_P -> /Serial/TX_A
- U3 pad 7: /Quadenc/A_IN_N -> /Serial/TX_B
- U4 pad 1: /Quadenc/A_IN_N -> unconnected-(U4-I/O1-Pad1)
- U4 pad 3: /Quadenc/A_IN_P -> unconnected-(U4-I/O2-Pad3)
- U4 pad 4: /Quadenc/B_IN_N -> Net-(U1-B)
- U4 pad 6: /Quadenc/B_IN_P -> Net-(U1-A)
- U5 pad 1: unconnected-(U5-I/O1-Pad1) -> /Serial/TX_A
- U5 pad 3: unconnected-(U5-I/O2-Pad3) -> /Serial/TX_B
- U5 pad 4: /Quadenc/Z_IN_N -> /Serial/RX_B
- U5 pad 6: /Quadenc/Z_IN_P -> /Serial/RX_A
- U6 pad 1: /Quadenc1/B -> Net-(D4-A1)
- U6 pad 2: GND -> Net-(U6A--)
- U6 pad 3: GND -> Net-(U6A-+)
- U6 pad 4: unconnected-(U6-DI-Pad4) -> GND
- U6 pad 5: GND -> Net-(U6B-+)
- U6 pad 6: /Quadenc1/B_IN_P -> Net-(U6B--)
- U6 pad 7: /Quadenc1/B_IN_N -> Net-(D2-A1)
- U6 pad 8: +3V3 -> Net-(U6C-V+)
Routing:
- net +3V3: track 467.1 -> 259.8 mm, vias 36 -> 17
- net +5V: track 247.2 -> 91.4 mm, vias 5 -> 1
- net GND: track 144.2 -> 35.9 mm, vias 163 -> 22
- net +24V: track 2.54 -> 80.2 mm, vias 0 -> 3
- net /Quadenc3/A: track 75.2 -> 0.00 mm, vias 1 -> 0
- net /Quadenc3/B: track 73.2 -> 0.00 mm, vias 1 -> 0
- net /Quadenc3/Z: track 71.5 -> 0.00 mm, vias 1 -> 0
- net /Quadenc2/A: track 69.3 -> 0.00 mm, vias 1 -> 0
- net /Quadenc2/B: track 67.5 -> 0.00 mm, vias 1 -> 0
- net /Serial/SSERIAL_RX: track 0.00 -> 67.4 mm, vias 0 -> 2
- net /Serial/MODBUS_A: track 0.00 -> 66.1 mm, vias 0 -> 1
- net /Quadenc2/Z: track 65.6 -> 0.00 mm, vias 1 -> 0
- net /Analog outputs/PWM_A1: track 0.00 -> 65.3 mm, vias 0 -> 2
- net /Serial/MODBUS_B: track 0.00 -> 64.5 mm, vias 0 -> 1
- net /Quadenc1/Z: track 60.1 -> 0.00 mm
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Other:
- board text added: "rioctrl-spindle v1.0"
- board text removed: "rioctrl-quadenc4 v1.0"
