File: rioctrl-spindle/rioctrl-spindle.kicad_sch (KiCad schematic)
At the start: 1 part, among them J1 TERM-BLK-02x05

Commit message: rioctrl-spindle v1.0 release
Connections:
- no-connect marks 1 -> 4
Changed lines of the file:
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@@
 		(at 120.65 74.93)
+	)
+	(no_connect
+		(at 120.65 52.07)
+	)
+	(no_connect
+		(at 120.65 49.53)
+	)
+	(no_connect
+		(at 245.11 54.61)
 	)
 	(wire
